Commit message: feat: add hand && calibration

File: ros_gluon/gluon/urdf/gluon.urdf (robot description, URDF)
Before this commit: robot gluon, 8 links, 7 joints
Links:
- added link fake_hand; collision box size=0.055 0.05 0.035; visual box size=0.055 0.05 0.035
Joints:
- added joint hand_joint: type fixed, parent 6_Link, child fake_hand, origin xyz=0.08 0 0 rpy=0 0 0
